File: esp32-NaziBeforeStiching.kicad_pcb (KiCad board)
At the start: 2 copper layers, 39.1 x 68.8 mm, 77 parts, among them J1 USB_C_Receptacle_USB2.0_14P, J2 Conn_01x02_Pin, J3 Conn_01x18_Pin, J5 Conn_01x18_Pin, Q1 AO3401A, U1 AMS1117-3.3, U2 ESP32-S3, U3 MCP73831-2-OT, U4 W25Q128JVS, Y1 40MHz(10ppm)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

Commit message: pcb_init+gerbers
Parts:
- removed G***, Gdfd: LOGO, LOGO
- moved R22 1.38 mm to (198.9, 109.5)
- moved C24 1.03 mm to (203.3, 84.6)
- moved C13 0.84 mm to (206.4, 68.2)
- moved R12 0.76 mm to (203.0, 82.3)
- moved Y2 0.59 mm to (195.5, 74.4)
- moved R19 0.54 mm to (191.2, 93.1)
- moved C4 0.44 mm to (212.9, 70.6)
- moved AE1 0.34 mm to (213.4, 63.0)
- moved C27 0.22 mm to (193.2, 73.6)
- moved C29 0.14 mm to (193.6, 76.2)
- moved R15 0.13 mm to (211.6, 75.7)
- turned D2 to 90 degrees
Connections:
- D2 pad 1: +5V -> Net-(D2-K)
- D2 pad 2: Net-(D2-A) -> +5V
- R9 pad 1: Net-(D2-A) -> Net-(D2-K)
Routing:
- net GND: track 125.9 -> 0.00 mm, vias 236 -> 0
- net IO14: track 61.6 -> 39.0 mm, vias 4 -> 3
- net Net-(D2-K): track 0.00 -> 9.44 mm
- net Net-(D2-A): track 9.44 -> 0.00 mm
- net USB_D+: track 50.6 -> 52.7 mm
- net USB_D-: track 51.4 -> 53.4 mm
- net SPICS0: track 20.4 -> 18.6 mm
- net VDD_SPI: track 16.3 -> 14.5 mm
- net VDD_CPU: track 126.3 -> 124.6 mm
- net Net-(U2-SPICLK): track 12.9 -> 14.4 mm
- net +5V: track 52.3 -> 51.0 mm, vias 4 -> 3
- net SPIWP: track 13.6 -> 12.6 mm
- net TX: track 8.54 -> 7.76 mm
- net XTAL32P: track 6.51 -> 7.29 mm
- net IO46: track 20.8 -> 20.1 mm
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Other:
- board size 39.1 x 68.8 mm -> 37.1 x 68.8 mm
- board text removed: "+5V"
- board text removed: "GND"
- board text removed: "IO0"
- board text removed: "IO10"
- board text removed: "IO11"
- board text removed: "IO12"
- board text removed: "IO13"
- board text removed: "IO14"
- board text removed: "IO17"
- board text removed: "IO18"
- board text removed: "IO2"
- board text removed: "IO21"
- board text removed: "IO3"
- board text removed: "IO33"
- board text removed: "IO34"
- board text removed: "IO35"
- board text removed: "IO36"
- board text removed: "IO37"
- board text removed: "IO38"
- board text removed: "IO39"
- board text removed: "IO40"
- board text removed: "IO41"
- board text removed: "IO42"
- board text removed: "IO45"
- board text removed: "IO46"
- board text removed: "IO47"
- board text removed: "IO48"
- board text removed: "IO5"
- board text removed: "IO6"
- board text removed: "IO7"
- board text removed: "IO8"
- board text removed: "IO9"
- board text removed: "RX"
- board text removed: "TX"
- board text removed: "VBAT"
- board text removed: "VDD"
