File: esp32-Nazi.kicad_pcb (KiCad board)
At the start: 2 copper layers, 39.1 x 68.8 mm, 77 parts, among them J1 USB_C_Receptacle_USB2.0_14P, J2 Conn_01x02_Pin, J3 Conn_01x18_Pin, J5 Conn_01x18_Pin, Q1 AO3401A, U1 AMS1117-3.3, U2 ESP32-S3, U3 MCP73831-2-OT, U4 W25Q128JVS, Y1 40MHz(10ppm)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

Commit message: production
Parts:
- R22: value 200K -> 100K
- turned C26 to 90 degrees
Connections:
- C26 pad 1: GND -> EN
- C26 pad 2: EN -> GND
