File: esp32-Nazi.kicad_sch (KiCad schematic)
At the start: 75 parts, among them J1 USB_C_Receptacle_USB2.0_14P, J2 Conn_01x02_Pin, J3 Conn_01x18_Pin, J5 Conn_01x18_Pin, Q1 AO3401A, U1 AMS1117-3.3, U2 ESP32-S3, U3 MCP73831-2-OT, U4 W25Q128JVS, Y1 40MHz(10ppm)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

Commit message: pcb_init+gerbers
Connections:
- net +5V: now also D2.1 (K), J3.16 (Pin_16); no longer D2.2 (A)
- net VBAT: now also Q1.3 (D); no longer Q1.2 (S)
- net VDD_SPI: no longer C13.2, L1.2, U2.2 (VDD3P3), U2.3 (VDD3P3)
- net VSYS: now also Q1.2 (S); no longer Q1.3 (D)
- net at R9.1: now also D2.2 (A); no longer D2.1 (K)
- net 5V renamed GND
- net GND: no longer J3.16 (Pin_16)
- new net: C13.2, L1.2, U2.2 (VDD3P3), U2.3 (VDD3P3)
Other:
- moved on the sheet: D2, Q1

Commit message: production
Parts:
- BTN1, Flash1, Reset1: MNF PART NUMBER (none) -> C318884
- C10, C14, C15, C23, C3, C6, C7, C8: MNF PART NUMBER (none) -> C15525
- C11, C12, C13, C17, C19, C2, C25: MNF PART NUMBER (none) -> C1525
- C16, C24, C9: MNF PART NUMBER (none) -> C52923
- C18, C26: MNF PART NUMBER (none) -> C15195
- C20, C21: MNF PART NUMBER (none) -> C1548
- C27, C29, C4, C5: MNF PART NUMBER (none) -> C1547
- D1, D2, D3: MNF PART NUMBER (none) -> C2286
- D4: MNF PART NUMBER (none) -> C2480
- J1: MNF PART NUMBER (none) -> C19274016
- L1: MNF PART NUMBER (none) -> C77103
- L2: MNF PART NUMBER (none) -> C13595
- Q1: MNF PART NUMBER (none) -> C15127
- R1, R2: MNF PART NUMBER (none) -> C25905
- R10, R11, R12, R13, R14, R5: MNF PART NUMBER (none) -> C17168
- R15, R6, R8: MNF PART NUMBER (none) -> C25117
- R16, R18, R19: MNF PART NUMBER (none) -> C25744
- R17: MNF PART NUMBER (none) -> C4109
- R20, R21: MNF PART NUMBER (none) -> C25764
- R22: value 200K -> 100K; MNF PART NUMBER (none) -> C25741
- R3: MNF PART NUMBER (none) -> 470R
- R4: MNF PART NUMBER (none) -> C25105
- R9: MNF PART NUMBER (none) -> C11702
- U1: MNF PART NUMBER (none) -> C6186
- U2: MNF PART NUMBER (none) -> C2913196; PartNumber C2913192 -> (none)
- U3: MNF PART NUMBER (none) -> C424093
- U4: MNF PART NUMBER (none) -> C97521
- Y1: MNF PART NUMBER (none) -> C5261125
- Y2: MNF PART NUMBER (none) -> C32346
Connections:
- net EN: now also C26.1; no longer C26.2
- net GND: now also C26.2; no longer C26.1
Other:
- moved on the sheet: C26
